File: vt100-addon.brd (EAGLE design)
At the start: 78.7 x 83.8 mm, 19 parts, among them IC1 TL77005ACP, Q1 MOSFET-NCHANNELPTH2, U1 MAX232PTH

Commit message: More board refinements
Parts:
- C101, C102, C103, C104: value 0.1uf -> 1uf
- C302: value 0.1uf -> 22uF; device sparkfun:CAP-PTH-SMALL -> sparkfun:CPOL-RADIAL-100UF-25V
- R303, R304: value 560 -> 10K
- moved U$7 30.4 mm to (37.6, 61.6)
- moved C302 26.3 mm to (47.0, 18.4), turned to 180 degrees
- moved R101 0.52 mm to (14.0, 20.3)
Routing:
- net N$20: track 14.4 -> 32.6 mm
- net GND: track 19.0 -> 8.11 mm, vias 54 -> 23
- net BB_GND: track 139.7 -> 141.8 mm
- net N$22: track 52.0 -> 52.7 mm, vias 2 -> 1

Commit message: A bit more cleanup
Parts:
- moved U$7 0.51 mm to (38.1, 61.6)
Changed lines of the file:
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@@
 <setting verticaltext="up"/>
 </settings>
-<grid distance="0.001" unitdist="inch" unit="inch" style="lines" multiple="1" display="yes" altdistance="0.005" altunitdist="inch" altunit="inch"/>
+<grid distance="0.025" unitdist="inch" unit="inch" style="lines" multiple="1" display="yes" altdistance="0.005" altunitdist="inch" altunit="inch"/>
 <layers>
 <layer number="1" name="Top" color="4" fill="1" visible="yes" active="yes"/>
@@
 <attribute name="VALUE" x="2.54" y="9.906" size="1.27" layer="27" ratio="10"/>
 </element>
-<element name="U$7" library="sparkfun" package="OSHW-LOGO-L" value="OSHW-LOGOL" x="37.592" y="61.595"/>
+<element name="U$7" library="sparkfun" package="OSHW-LOGO-L" value="OSHW-LOGOL" x="38.1" y="61.595"/>
 <element name="C302" library="sparkfun" package="CPOL-RADIAL-100UF-25V" value="22uF" x="46.99" y="18.415" smashed="yes" rot="R180">
 <attribute name="VALUE" x="48.895" y="22.733" size="0.8128" layer="27" rot="R180"/>
