File: vt100-addon.sch (EAGLE design)
At the start: 19 parts, among them IC1 TL77005ACP, Q1 MOSFET-NCHANNELPTH2, U1 MAX232PTH

Commit message: More board refinements
Parts:
- C101, C102, C103, C104: value 0.1uf -> 1uf
- C302: value 0.1uf -> 22uF; device sparkfun:CAPPTH -> sparkfun:CAP_POLPTH1
- R303, R304: value 560 -> 10K
Connections:
- net GND: now also C302.-; no longer C302.2
- net N$20: now also C302.+; no longer C302.1
Changed lines of the file:
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@@
 <part name="U$2" library="custom" deviceset="STP_EDGE" device=""/>
 <part name="C105" library="sparkfun" deviceset="CAP" device="PTH" value="0.1uf"/>
-<part name="C101" library="sparkfun" deviceset="CAP" device="PTH" value="0.1uf"/>
-<part name="C102" library="sparkfun" deviceset="CAP" device="PTH" value="0.1uf"/>
-<part name="C104" library="sparkfun" deviceset="CAP" device="PTH" value="0.1uf"/>
-<part name="C103" library="sparkfun" deviceset="CAP" device="PTH" value="0.1uf"/>
+<part name="C101" library="sparkfun" deviceset="CAP" device="PTH" value="1uf"/>
+<part name="C102" library="sparkfun" deviceset="CAP" device="PTH" value="1uf"/>
+<part name="C104" library="sparkfun" deviceset="CAP" device="PTH" value="1uf"/>
+<part name="C103" library="sparkfun" deviceset="CAP" device="PTH" value="1uf"/>
 <part name="GND1" library="sparkfun" deviceset="GND" device=""/>
 <part name="GND2" library="sparkfun" deviceset="GND" device=""/>
@@
 <part name="U$6" library="sparkfun" deviceset="5V" device=""/>
 <part name="C301" library="sparkfun" deviceset="CAP" device="PTH" value="0.1uf"/>
-<part name="C302" library="sparkfun" deviceset="CAP" device="PTH" value="0.1uf"/>
 <part name="C303" library="sparkfun" deviceset="CAP" device="PTH" value="0.1uf"/>
 <part name="GND12" library="sparkfun" deviceset="GND" device=""/>
 <part name="R302" library="sparkfun" deviceset="RESISTOR" device="PTH-1/4W" value="560"/>
-<part name="R303" library="sparkfun" deviceset="RESISTOR" device="PTH-1/4W" value="560"/>
-<part name="R304" library="sparkfun" deviceset="RESISTOR" device="PTH-1/4W" value="560"/>
+<part name="R303" library="sparkfun" deviceset="RESISTOR" device="PTH-1/4W" value="10K"/>
+<part name="R304" library="sparkfun" deviceset="RESISTOR" device="PTH-1/4W" value="10K"/>
 <part name="R301" library="sparkfun" deviceset="RESISTOR" device="PTH-1/4W" value="10k"/>
 <part name="Q1" library="sparkfun" deviceset="MOSFET-NCHANNEL" device="PTH2"/>
 <part name="FRAME1" library="sparkfun" deviceset="FRAME-LETTER" device=""/>
 <part name="U$7" library="sparkfun" deviceset="OSHW-LOGO" device="L"/>
+<part name="C302" library="sparkfun" deviceset="CAP_POL" device="PTH1" value="22uF"/>
 </parts>
 <sheets>
@@
 <instance part="U$6" gate="G$1" x="-58.42" y="-45.72"/>
 <instance part="C301" gate="G$1" x="-58.42" y="-60.96" rot="R180"/>
-<instance part="C302" gate="G$1" x="-50.8" y="-66.04" rot="R270"/>
 <instance part="C303" gate="G$1" x="12.7" y="-73.66" rot="R180"/>
 <instance part="GND12" gate="1" x="12.7" y="-86.36"/>
@@
 <instance part="FRAME1" gate="G$2" x="81.28" y="-91.44"/>
 <instance part="U$7" gate="G$1" x="66.04" y="-78.74"/>
+<instance part="C302" gate="G$1" x="-48.26" y="-66.04" rot="R270"/>
 </instances>
 <busses>
@@
 <wire x1="12.7" y1="-78.74" x2="12.7" y2="-81.28" width="0.1524" layer="91"/>
 <pinref part="C301" gate="G$1" pin="1"/>
-<pinref part="C302" gate="G$1" pin="2"/>
 <wire x1="12.7" y1="-81.28" x2="12.7" y2="-83.82" width="0.1524" layer="91"/>
-<wire x1="-53.34" y1="-66.04" x2="-58.42" y2="-66.04" width="0.1524" layer="91"/>
 <wire x1="-58.42" y1="-66.04" x2="-58.42" y2="-81.28" width="0.1524" layer="91"/>
-<junction x="-58.42" y="-66.04"/>
 <wire x1="-58.42" y1="-81.28" x2="12.7" y2="-81.28" width="0.1524" layer="91"/>
 <junction x="12.7" y="-81.28"/>
@@
 <wire x1="35.56" y1="-81.28" x2="20.32" y2="-81.28" width="0.1524" layer="91"/>
 <junction x="20.32" y="-81.28"/>
+<pinref part="C302" gate="G$1" pin="-"/>
+<wire x1="-53.34" y1="-66.04" x2="-58.42" y2="-66.04" width="0.1524" layer="91"/>
+<junction x="-58.42" y="-66.04"/>
 </segment>
 </net>
@@
 </segment>
 </net>
-<net name="N$20" class="0">
-<segment>
-<pinref part="R302" gate="G$1" pin="2"/>
-<pinref part="C302" gate="G$1" pin="1"/>
-<wire x1="-43.18" y1="-66.04" x2="-45.72" y2="-66.04" width="0.1524" layer="91"/>
-</segment>
-</net>
 <net name="N$21" class="0">
 <segment>
@@
 </segment>
 </net>
+<net name="N$20" class="0">
+<segment>
+<pinref part="R302" gate="G$1" pin="2"/>
+<pinref part="C302" gate="G$1" pin="+"/>
+<wire x1="-43.18" y1="-66.04" x2="-45.72" y2="-66.04" width="0.1524" layer="91"/>
+</segment>
+</net>
